Commit message: added gazebo PID controllers, reversed left and right wheels.

File: urdf/simple_robot_custom_ctlr.xacro (robot description, xacro)
@@ -109,5 +109,5 @@
         <parent link="chassis"/>
         <child link="left_wheel"/>
-        <origin xyz="-0.1 0.13 0" rpy="0 1.5707 1.5707"/>
+        <origin xyz="-0.1 -0.13 0" rpy="0 1.5707 1.5707"/>
         <axis xyz="0 0 1"/>
         <calibration rising="0.0"/>
@@ -119,5 +119,5 @@
         <parent link="chassis"/>
         <child link="right_wheel"/>
-        <origin xyz="-0.1 -0.13 0" rpy="0 1.5707 1.5707"/>
+        <origin xyz="-0.1 0.13 0" rpy="0 1.5707 1.5707"/>
         <axis xyz="0 0 1"/>
         <calibration rising="0.0"/>

Commit message: Including in git matlab controller template

File: urdf/simple_robot_custom_ctlr.xacro (robot description, xacro)
@@ -109,5 +109,5 @@
         <parent link="chassis"/>
         <child link="left_wheel"/>
-        <origin xyz="-0.1 -0.13 0" rpy="0 1.5707 1.5707"/>
+        <origin xyz="-0.1 -0.13 0" rpy="0 -1.5707 1.5707"/>
         <axis xyz="0 0 1"/>
         <calibration rising="0.0"/>
@@ -119,5 +119,5 @@
         <parent link="chassis"/>
         <child link="right_wheel"/>
-        <origin xyz="-0.1 0.13 0" rpy="0 1.5707 1.5707"/>
+        <origin xyz="-0.1 0.13 0" rpy="0 -1.5707 1.5707"/>
         <axis xyz="0 0 1"/>
         <calibration rising="0.0"/>

Commit message: Updated weights and inertias for a more realistic movement

File: urdf/simple_robot_custom_ctlr.xacro (robot description, xacro)
@@ -16,6 +16,6 @@
     <link name="chassis">
         <inertial>
-            <mass value="1"/>
-            <inertia ixx="0.004" ixy="0.0" ixz="0.0" iyy="0.004" iyz="0.0" izz="0.002"/>
+            <mass value="20"/>
+            <inertia ixx="1" ixy="0.0" ixz="0.0" iyy="1" iyz="0.0" izz="1"/>
         </inertial>
         <collision name='collision'>
@@ -57,6 +57,6 @@
     <link name="left_wheel">
         <inertial>
-            <mass value=".5"/>
-            <inertia ixx="1" ixy="0.0" ixz="0.0" iyy="1" iyz="0.0" izz="1"/>
+            <mass value=".15"/>
+            <inertia ixx="0.1" ixy="0.0" ixz="0.0" iyy="0.1" iyz="0.0" izz="0.1"/>
         </inertial>
         <pose>0.1 0.13 0.1 0 1.5707 1.5707</pose>
@@ -75,6 +75,6 @@
     <link name="right_wheel">
         <inertial>
-            <mass value=".5"/>
-            <inertia ixx="1" ixy="0.0" ixz="0.0" iyy="1" iyz="0.0" izz="1"/>
+            <mass value=".15"/>
+            <inertia ixx="0.1" ixy="0.0" ixz="0.0" iyy="0.1" iyz="0.0" izz="0.1"/>
         </inertial>
         <pose>0.1 0.13 0.1 0 1.5707 1.5707</pose>
